File: sch/uwm_esp32/uwm_esp32.kicad_sch (KiCad schematic)
At the start: 25 parts, among them SW1 Sleep Button, SW2 Mode Button, U1 XIAO_ESP32C3, U2 DWM3000TR13

Commit message: Add IRQ pull-up to ESP32 schematic
Replace the mode button with a 100k IRQ pull-up, add a test point, and set the capacitor values to 10uF and 100nF.
Parts:
- removed SW2: Mode Button, Package_DFN_QFN:TDFN-12_2x3mm_P0.5mm, symbol Switch:SW_Push
- added R7: 100k, symbol Device:R
- added TP8: TestPoint, symbol Connector:TestPoint
- C1: value C_Small -> 100n
- C2: value C_Small -> 10u
Connections:
- net GND: now also R7.2
- net IRQ: now also U1.11 (D10), R7.1; no longer U1.1 (D0)
- new net: TP8.1, U1.1 (D0)
Changed lines of the file:
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@@
 	)
 	(junction
-		(at 100.33 74.93)
+		(at 210.82 105.41)
 		(diameter 0)
 		(color 0 0 0 0)
 	)
 	(junction
-		(at 210.82 105.41)
+		(at 215.9 48.26)
 		(diameter 0)
 		(color 0 0 0 0)
 	)
 	(junction
-		(at 215.9 48.26)
+		(at 100.33 72.39)
 		(diameter 0)
 		(color 0 0 0 0)
@@
 	(wire
 		(pts
-			(xy 118.11 72.39) (xy 118.11 74.93)
-		)
-		(stroke
-			(width 0)
-			(type default)
-		)
-	)
-	(wire
-		(pts
 			(xy 240.03 49.53) (xy 240.03 48.26)
 		)
@@
 	(wire
 		(pts
-			(xy 100.33 72.39) (xy 100.33 74.93)
+			(xy 100.33 72.39) (xy 100.33 76.2)
 		)
 		(stroke
@@
 	(wire
 		(pts
-			(xy 100.33 74.93) (xy 100.33 76.2)
+			(xy 53.34 59.69) (xy 62.23 59.69)
 		)
 		(stroke
@@
 	(wire
 		(pts
-			(xy 53.34 59.69) (xy 62.23 59.69)
+			(xy 195.58 99.06) (xy 198.12 99.06)
 		)
 		(stroke
@@
 	(wire
 		(pts
-			(xy 195.58 99.06) (xy 198.12 99.06)
+			(xy 55.88 49.53) (xy 50.8 49.53)
 		)
 		(stroke
@@
 	(wire
 		(pts
-			(xy 104.14 72.39) (xy 107.95 72.39)
+			(xy 97.79 59.69) (xy 106.68 59.69)
 		)
 		(stroke
@@
 	(wire
 		(pts
-			(xy 97.79 59.69) (xy 106.68 59.69)
+			(xy 212.09 71.12) (xy 220.98 71.12)
 		)
 		(stroke
@@
 	(wire
 		(pts
-			(xy 212.09 71.12) (xy 220.98 71.12)
+			(xy 55.88 49.53) (xy 55.88 54.61)
 		)
 		(stroke
@@
 	(wire
 		(pts
-			(xy 104.14 64.77) (xy 104.14 72.39)
-		)
-		(stroke
-			(width 0)
-			(type default)
-		)
-	)
-	(wire
-		(pts
 			(xy 215.9 50.8) (xy 215.9 48.26)
 		)
@@
 	(wire
 		(pts
-			(xy 78.74 96.52) (xy 78.74 100.33)
+			(xy 100.33 72.39) (xy 104.14 72.39)
 		)
 		(stroke
@@
 	(wire
 		(pts
-			(xy 210.82 99.06) (xy 210.82 105.41)
+			(xy 78.74 96.52) (xy 78.74 100.33)
 		)
 		(stroke
@@
 	(wire
 		(pts
-			(xy 224.79 49.53) (xy 240.03 49.53)
+			(xy 210.82 99.06) (xy 210.82 105.41)
 		)
 		(stroke
@@
 	(wire
 		(pts
-			(xy 118.11 74.93) (xy 100.33 74.93)
+			(xy 224.79 49.53) (xy 240.03 49.53)
 		)
 		(stroke
@@
 	(wire
 		(pts
-			(xy 53.34 54.61) (xy 62.23 54.61)
+			(xy 55.88 54.61) (xy 62.23 54.61)
 		)
 		(stroke
@@
 		)
 	)
-	(label "IRQ"
-		(at 53.34 54.61 0)
+	(label "RSTn"
+		(at 99.06 54.61 0)
 		(effects
 			(font
@@
 		)
 	)
-	(label "RSTn"
-		(at 99.06 54.61 0)
+	(label "SPICSn"
+		(at 213.36 63.5 0)
 		(effects
 			(font
@@
 		)
 	)
-	(label "SPICSn"
-		(at 213.36 63.5 0)
+	(label "SPIMISO"
+		(at 53.34 59.69 0)
 		(effects
 			(font
@@
 		)
 	)
-	(label "SPIMISO"
-		(at 53.34 59.69 0)
+	(label "IRQ"
+		(at 99.06 64.77 0)
 		(effects
 			(font
@@
 			)
 		)
-		(property "Value" "C_Small"
+		(property "Value" "10u"
 			(at 242.57 46.9899 0)
 			(show_name no)
@@
 	)
 	(symbol
+		(lib_id "Device:R")
+		(at 104.14 68.58 0)
+		(unit 1)
+		(body_style 1)
+		(exclude_from_sim no)
+		(in_bom yes)
+		(on_board yes)
+		(in_pos_files yes)
+		(dnp no)
+		(fields_autoplaced yes)
+		(property "Reference" "R7"
+			(at 106.68 67.3099 0)
+			(show_name no)
+			(do_not_autoplace no)
+			(effects
+				(font
+					(size 1.27 1.27)
+				)
+				(justify left)
+			)
+		)
+		(property "Value" "100k"
+			(at 106.68 69.8499 0)
+			(show_name no)
+			(do_not_autoplace no)
+			(effects
+				(font
+					(size 1.27 1.27)
+				)
+				(justify left)
+			)
+		)
+		(property "Footprint" ""
+			(at 102.362 68.58 90)
+			(hide yes)
+			(show_name no)
+			(do_not_autoplace no)
+			(effects
+				(font
+					(size 1.27 1.27)
+				)
+			)
+		)
+		(property "Datasheet" ""
+			(at 104.14 68.58 0)
+			(hide yes)
+			(show_name no)
+			(do_not_autoplace no)
+			(effects
+				(font
+					(size 1.27 1.27)
+				)
+			)
+		)
+		(property "Description" "Resistor"
+			(at 104.14 68.58 0)
+			(hide yes)
+			(show_name no)
+			(do_not_autoplace no)
+			(effects
+				(font
+					(size 1.27 1.27)
+				)
+			)
+		)
+		(pin "2"
+		)
+		(pin "1"
+		)
+		(instances
+			(project "uwm_esp32"
+				(path "/a6d4bd55-872a-4f27-8506-f77c397732a2"
+					(reference "R7")
+					(unit 1)
+				)
+			)
+		)
+	)
+	(symbol
 		(lib_id "power:GND")
 		(at 223.52 85.09 0)
@@
 	(symbol
 		(lib_id "Connector:TestPoint")
+		(at 50.8 49.53 90)
+		(unit 1)
+		(body_style 1)
+		(exclude_from_sim no)
+		(in_bom yes)
+		(on_board yes)
+		(in_pos_files yes)
+		(dnp no)
+		(property "Reference" "TP8"
+			(at 46.99 51.054 90)
+			(show_name no)
+			(do_not_autoplace no)
+			(effects
+				(font
+					(size 1.27 1.27)
+				)
+			)
+		)
+		(property "Value" "TestPoint"
+			(at 41.148 49.53 90)
+			(show_name no)
+			(do_not_autoplace no)
+			(effects
+				(font
+					(size 1.27 1.27)
+				)
+			)
+		)
+		(property "Footprint" ""
+			(at 50.8 44.45 0)
+			(hide yes)
+			(show_name no)
+			(do_not_autoplace no)
+			(effects
+				(font
+					(size 1.27 1.27)
+				)
+			)
+		)
+		(property "Datasheet" ""
+			(at 50.8 44.45 0)
+			(hide yes)
+			(show_name no)
+			(do_not_autoplace no)
+			(effects
+				(font
+					(size 1.27 1.27)
+				)
+			)
+		)
+		(property "Description" "test point"
+			(at 50.8 49.53 0)
+			(hide yes)
+			(show_name no)
+			(do_not_autoplace no)
+			(effects
+				(font
+					(size 1.27 1.27)
+				)
+			)
+		)
+		(pin "1"
+		)
+		(instances
+			(project "uwm_esp32"
+				(path "/a6d4bd55-872a-4f27-8506-f77c397732a2"
+					(reference "TP8")
+					(unit 1)
+				)
+			)
+		)
+	)
+	(symbol
+		(lib_id "Connector:TestPoint")
 		(at 106.68 62.23 270)
 		(unit 1)
@@
 	)
 	(symbol
-		(lib_id "Switch:SW_Push")
-		(at 113.03 72.39 0)
-		(unit 1)
-		(body_style 1)
-		(exclude_from_sim no)
-		(in_bom yes)
-		(on_board yes)
-		(in_pos_files yes)
-		(dnp no)
-		(property "Reference" "SW2"
-			(at 108.712 69.342 0)
-			(show_name no)
-			(do_not_autoplace no)
-			(effects
-				(font
-					(size 1.27 1.27)
-				)
-			)
-		)
-		(property "Value" "Mode Button"
-			(at 111.506 73.914 0)
-			(show_name no)
-			(do_not_autoplace no)
-			(effects
-				(font
-					(size 1.27 1.27)
-				)
-			)
-		)
-		(property "Footprint" "Package_DFN_QFN:TDFN-12_2x3mm_P0.5mm"
-			(at 113.03 67.31 0)
-			(hide yes)
-			(show_name no)
-			(do_not_autoplace no)
-			(effects
-				(font
-					(size 1.27 1.27)
-				)
-			)
-		)
-		(property "Datasheet" ""
-			(at 113.03 67.31 0)
-			(hide yes)
-			(show_name no)
-			(do_not_autoplace no)
-			(effects
-				(font
-					(size 1.27 1.27)
-				)
-			)
-		)
-		(property "Description" "Push button switch, generic, two pins"
-			(at 113.03 72.39 0)
-			(hide yes)
-			(show_name no)
-			(do_not_autoplace no)
-			(effects
-				(font
-					(size 1.27 1.27)
-				)
-			)
-		)
-		(pin "2"
-		)
-		(pin "1"
-		)
-		(instances
-			(project "uwm_esp32"
-				(path "/a6d4bd55-872a-4f27-8506-f77c397732a2"
-					(reference "SW2")
-					(unit 1)
-				)
-			)
-		)
-	)
-	(symbol
 		(lib_id "Device:C_Small")
 		(at 224.79 45.72 0)
@@
 			)
 		)
-		(property "Value" "C_Small"
+		(property "Value" "100n"
 			(at 227.33 46.9899 0)
 			(show_name no)

Commit message: Add sleep button pull-up circuitry
Add a 10 kΩ resistor and +3V3 connection, reposition the sleep button and TP8, and update the related wiring and labels.
Parts:
- added R8: 10k, symbol Device:R
Connections:
- net +3V3: now also R8.1
- net ModeLED: now also U1.7 (TX_D6); no longer U1.8 (RX_D7)
- net RSTn: now also U1.8 (RX_D7); no longer U1.7 (TX_D6)
- net at SW1.2, U1.2 (D1): now also R8.2
Other:
- moved on the sheet: SW1, TP8
Changed lines of the file:
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@@
 	)
 	(junction
+		(at 46.99 57.15)
+		(diameter 0)
+		(color 0 0 0 0)
+	)
+	(junction
 		(at 100.33 72.39)
 		(diameter 0)
@@
 	(wire
 		(pts
-			(xy 55.88 49.53) (xy 50.8 49.53)
+			(xy 60.96 48.26) (xy 58.42 48.26)
+		)
+		(stroke
+			(width 0)
+			(type default)
+		)
+	)
+	(wire
+		(pts
+			(xy 97.79 57.15) (xy 106.68 57.15)
 		)
 		(stroke
@@
 	(wire
 		(pts
-			(xy 53.34 57.15) (xy 62.23 57.15)
+			(xy 44.45 57.15) (xy 46.99 57.15)
 		)
 		(stroke
@@
 	(wire
 		(pts
-			(xy 55.88 49.53) (xy 55.88 54.61)
+			(xy 60.96 48.26) (xy 60.96 54.61)
 		)
 		(stroke
@@
 	(wire
 		(pts
-			(xy 43.18 57.15) (xy 38.1 57.15)
+			(xy 34.29 57.15) (xy 29.21 57.15)
 		)
 		(stroke
@@
 	(wire
 		(pts
-			(xy 38.1 57.15) (xy 38.1 58.42)
+			(xy 29.21 57.15) (xy 29.21 58.42)
 		)
 		(stroke
@@
 	(wire
 		(pts
+			(xy 46.99 48.26) (xy 46.99 49.53)
+		)
+		(stroke
+			(width 0)
+			(type default)
+		)
+	)
+	(wire
+		(pts
 			(xy 63.5 33.02) (xy 63.5 29.21)
 		)
@@
 	(wire
 		(pts
+			(xy 46.99 57.15) (xy 62.23 57.15)
+		)
+		(stroke
+			(width 0)
+			(type default)
+		)
+	)
+	(wire
+		(pts
 			(xy 210.82 120.65) (xy 210.82 118.11)
 		)
@@
 	(wire
 		(pts
-			(xy 55.88 54.61) (xy 62.23 54.61)
-		)
-		(stroke
-			(width 0)
-			(type default)
-		)
-	)
-	(wire
-		(pts
-			(xy 97.79 57.15) (xy 106.68 57.15)
+			(xy 60.96 54.61) (xy 62.23 54.61)
 		)
 		(stroke
@@
 	)
 	(label "RSTn"
-		(at 99.06 54.61 0)
+		(at 99.06 57.15 0)
 		(effects
 			(font
@@
 	)
 	(label "ModeLED"
-		(at 99.06 57.15 0)
+		(at 99.06 54.61 0)
 		(effects
 			(font
@@
 	(symbol
 		(lib_id "Switch:SW_Push")
-		(at 48.26 57.15 0)
+		(at 39.37 57.15 0)
 		(unit 1)
 		(body_style 1)
@@
 		(dnp no)
 		(property "Reference" "SW1"
-			(at 43.942 54.102 0)
+			(at 35.052 54.102 0)
 			(show_name no)
 			(do_not_autoplace no)
@@
 		)
 		(property "Value" "Sleep Button"
-			(at 46.482 59.436 0)
+			(at 37.592 59.436 0)
 			(show_name no)
 			(do_not_autoplace no)
@@
 		)
 		(property "Footprint" "Package_DFN_QFN:TDFN-12_2x3mm_P0.5mm"
-			(at 48.26 52.07 0)
+			(at 39.37 52.07 0)
 			(hide yes)
 			(show_name no)
@@
 		)
 		(property "Datasheet" ""
-			(at 48.26 52.07 0)
+			(at 39.37 52.07 0)
 			(hide yes)
 			(show_name no)
@@
 		)
 		(property "Description" "Push button switch, generic, two pins"
-			(at 48.26 57.15 0)
+			(at 39.37 57.15 0)
 			(hide yes)
 			(show_name no)
@@
 	)
 	(symbol
+		(lib_id "power:+3V3")
+		(at 46.99 48.26 0)
+		(unit 1)
+		(body_style 1)
+		(exclude_from_sim no)
+		(in_bom yes)
+		(on_board yes)
+		(in_pos_files yes)
+		(dnp no)
+		(fields_autoplaced yes)
+		(property "Reference" "#PWR08"
+			(at 46.99 52.07 0)
+			(hide yes)
+			(show_name no)
+			(do_not_autoplace no)
+			(effects
+				(font
+					(size 1.27 1.27)
+				)
+			)
+		)
+		(property "Value" "+3V3"
+			(at 46.99 43.18 0)
+			(show_name no)
+			(do_not_autoplace no)
+			(effects
+				(font
+					(size 1.27 1.27)
+				)
+			)
+		)
+		(property "Footprint" ""
+			(at 46.99 48.26 0)
+			(hide yes)
+			(show_name no)
+			(do_not_autoplace no)
+			(effects
+				(font
+					(size 1.27 1.27)
+				)
+			)
+		)
+		(property "Datasheet" ""
+			(at 46.99 48.26 0)
+			(hide yes)
+			(show_name no)
+			(do_not_autoplace no)
+			(effects
+				(font
+					(size 1.27 1.27)
+				)
+			)
+		)
+		(property "Description" "Power symbol creates a global label with name \"+3V3\""
+			(at 46.99 48.26 0)
+			(hide yes)
+			(show_name no)
+			(do_not_autoplace no)
+			(effects
+				(font
+					(size 1.27 1.27)
+				)
+			)
+		)
+		(pin "1"
+		)
+		(instances
+			(project "uwm_esp32"
+				(path "/a6d4bd55-872a-4f27-8506-f77c397732a2"
+					(reference "#PWR08")
+					(unit 1)
+				)
+			)
+		)
+	)
+	(symbol
 		(lib_id "Device:R")
 		(at 104.14 68.58 0)
@@
 	(symbol
 		(lib_id "Connector:TestPoint")
-		(at 50.8 49.53 90)
+		(at 58.42 48.26 90)
 		(unit 1)
 		(body_style 1)
@@
 		(dnp no)
 		(property "Reference" "TP8"
-			(at 46.99 51.054 90)
+			(at 55.372 50.292 90)
 			(show_name no)
 			(do_not_autoplace no)
@@
 		)
 		(property "Value" "TestPoint"
-			(at 41.148 49.53 90)
+			(at 55.88 45.974 90)
 			(show_name no)
 			(do_not_autoplace no)
@@
 		)
 		(property "Footprint" ""
-			(at 50.8 44.45 0)
+			(at 58.42 43.18 0)
 			(hide yes)
 			(show_name no)
@@
 		)
 		(property "Datasheet" ""
-			(at 50.8 44.45 0)
+			(at 58.42 43.18 0)
 			(hide yes)
 			(show_name no)
@@
 		)
 		(property "Description" "test point"
-			(at 50.8 49.53 0)
+			(at 58.42 48.26 0)
 			(hide yes)
 			(show_name no)
@@
 	)
 	(symbol
+		(lib_id "Device:R")
+		(at 46.99 53.34 0)
+		(unit 1)
+		(body_style 1)
+		(exclude_from_sim no)
+		(in_bom yes)
+		(on_board yes)
+		(in_pos_files yes)
+		(dnp no)
+		(fields_autoplaced yes)
+		(property "Reference" "R8"
+			(at 49.53 52.0699 0)
+			(show_name no)
+			(do_not_autoplace no)
+			(effects
+				(font
+					(size 1.27 1.27)
+				)
+				(justify left)
+			)
+		)
+		(property "Value" "10k"
+			(at 49.53 54.6099 0)
+			(show_name no)
+			(do_not_autoplace no)
+			(effects
+				(font
+					(size 1.27 1.27)
+				)
+				(justify left)
+			)
+		)
+		(property "Footprint" ""
+			(at 45.212 53.34 90)
+			(hide yes)
+			(show_name no)
+			(do_not_autoplace no)
+			(effects
+				(font
+					(size 1.27 1.27)
+				)
+			)
+		)
+		(property "Datasheet" ""
+			(at 46.99 53.34 0)
+			(hide yes)
+			(show_name no)
+			(do_not_autoplace no)
+			(effects
+				(font
+					(size 1.27 1.27)
+				)
+			)
+		)
+		(property "Description" "Resistor"
+			(at 46.99 53.34 0)
+			(hide yes)
+			(show_name no)
+			(do_not_autoplace no)
+			(effects
+				(font
+					(size 1.27 1.27)
+				)
+			)
+		)
+		(pin "2"
+		)
+		(pin "1"
+		)
+		(instances
+			(project "uwm_esp32"
+				(path "/a6d4bd55-872a-4f27-8506-f77c397732a2"
+					(reference "R8")
+					(unit 1)
+				)
+			)
+		)
+	)
+	(symbol
 		(lib_id "Device:C_Small")
 		(at 224.79 45.72 0)
@@
 	(symbol
 		(lib_id "power:GND")
-		(at 38.1 58.42 0)
+		(at 29.21 58.42 0)
 		(unit 1)
 		(body_style 1)
@@
 		(fields_autoplaced yes)
 		(property "Reference" "#PWR01"
-			(at 38.1 64.77 0)
+			(at 29.21 64.77 0)
 			(hide yes)
 			(show_name no)
@@
 		)
 		(property "Value" "GND"
-			(at 38.1 63.5 0)
+			(at 29.21 63.5 0)
 			(show_name no)
 			(do_not_autoplace no)
@@
 		)
 		(property "Footprint" ""
-			(at 38.1 58.42 0)
+			(at 29.21 58.42 0)
 			(hide yes)
 			(show_name no)
@@
 		)
 		(property "Datasheet" ""
-			(at 38.1 58.42 0)
+			(at 29.21 58.42 0)
 			(hide yes)
 			(show_name no)
@@
 		)
 		(property "Description" "Power symbol creates a global label with name \"GND\" , ground"
-			(at 38.1 58.42 0)
+			(at 29.21 58.42 0)
 			(hide yes)
 			(show_name no)

Commit message: Add ESP32 and DWM edge headers
Replace test points with six-pin edge headers, connect the ESP32-C3 and DWM3000 signals, and update the PCB layout with the module and supporting components.
Parts:
- removed TP1, TP2, TP3, TP4, TP5, TP6, TP7, TP8: TestPoint, symbol Connector:TestPoint
- added J1: ESP32 Edge Header, Connector_PinHeader_2.54mm:PinHeader_1x06_P2.54mm_Vertical, symbol Connector:Conn_01x06_Pin
- added J2: DWM Edge Header, Connector_PinHeader_2.54mm:PinHeader_1x06_P2.54mm_Vertical, symbol Connector:Conn_01x06_Pin
- C1, C2: footprint (none) -> Capacitor_SMD:C_0805_2012Metric_Pad1.18x1.45mm_HandSolder
- D1, D2, D3, D4, D5, D6: footprint (none) -> LED_SMD:LED_0805_2012Metric_Pad1.15x1.40mm_HandSolder
- R1, R2, R3, R4, R5, R6, R7, R8: footprint (none) -> Resistor_SMD:R_0805_2012Metric_Pad1.20x1.40mm_HandSolder
- SW1: footprint Package_DFN_QFN:TDFN-12_2x3mm_P0.5mm -> Button_Switch_SMD:SW_SPST_Omron_B3FS-101xP
Connections:
- net +3V3: now also J1.1 (Pin_1)
- net EXTON: now also J2.2 (Pin_2)
- net GND: now also J1.3 (Pin_3), J1.6 (Pin_6), J2.1 (Pin_1)
- net GPIO4: now also J2.4 (Pin_4)
- net SPIPHA: now also J2.5 (Pin_5)
- net SPIPOL: now also J2.6 (Pin_6)
- net SYNC: now also J2.3 (Pin_3)
- net D0: now reaches U1.1 (D0)
- net D0: now also J1.2 (Pin_2)
- net D9: now reaches U1.10 (D9)
- net D9: now also J1.5 (Pin_5)
- net D8: now reaches U1.9 (D8)
- net D8: now also J1.4 (Pin_4)
